Commit message: organised files/changing names

File: urdf/robot_core.xacro (robot description, xacro)
@@ -54,5 +54,5 @@
                 <box size="${chassis_length} ${chassis_width} ${chassis_height}"/>
             </geometry>
-            <material name="orange"/>
+            <material name="white"/>
         </visual>
         <collision>

File: urdf/sensors/lidar.xacro (robot description, xacro)
@@ -11,5 +11,5 @@
                 <cylinder radius="0.05" length="0.04"/>
             </geometry>
-            <material name="black"/>
+            <material name="red"/>
         </visual>
         <visual>
